File: kvm/kvm.kicad_sch (KiCad schematic)
At the start: 61 parts, among them J1 USB4110-GF-A, J2 USB4110-GF-A, J3 USB_A_Stacked, J4 USB_A_Stacked, Q1 Q_PMOS_GSD, SW1 SW_DPDT_x2, U1 SRV05-4, U2 LTC4412xS6, U3 FSUSB42MUX, U4 GL850G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

Commit message: added gerber files
Other:
- note added: "3.3V Rail"
- note added: "Clock"
- note added: "Hub Peripherie"
- note added: "Input ESD Protection"
- note added: "LED Indicator"
- note added: "Output ESD Protection"
- note added: "Overcurrent protection"
- note added: "Power Distribution"
- note added: "Reset"
- note added: "USB Outputs"
- note added: "USB Switch"
- note added: "USB-C Inputs"
- note added: "USB-Hub Controller"
- moved on the sheet: C1, C10, C11, C12, C13, C14, C15, C16, C17, C18, C19, C2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

Commit message: added buy links
Parts:
- C10: MouserLink (none) -> https://www.mouser.at/ProductDetail/Taiyo-Yuden/LMK212ABJ10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
- C11, C12, C14, C17, C18, C21, C4, C5: MouserLink (none) -> https://www.mouser.at/ProductDetail/TDK/C0603X5R1E104K030BB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
- C15, C16, C6, C7: MouserLink (none) -> https://www.mouser.at/ProductDetail/Panasonic/EEU-FR1C101?q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
- C20: MouserLink (none) -> https://www.mouser.at/ProductDetail/KYOCERA-AVX/06033A330FA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
- D1: MouserLink (none) -> https://www.mouser.at/ProductDetail/ROHM-Semiconductor/RB16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
- D2: MouserLink (none) -> https://www.mouser.at/ProductDetail/Kingbright/APTD2012LSUR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
- F1, F2, F3, F4: MouserLink (none) -> https://www.mouser.at/ProductDetail/Littelfuse/1206L050YR?q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
- J1, J2: MouserLink (none) -> https://www.mouser.at/ProductDetail/GCT/USB4110-GF-A?qs=KUo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
- J3, J4: MouserLink (none) -> https://www.mouser.at/ProductDetail/Wurth-Elektronik/614008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
- Q1: MouserLink (none) -> https://www.mouser.at/ProductDetail/Toshiba/SSM3J372RLXHF?q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
- U1, U5, U6: MouserLink (none) -> https://www.mouser.at/ProductDetail/Littelfuse/SRV05-4HTG-D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
- U2: MouserLink (none) -> https://www.mouser.at/ProductDetail/Analog-Devices/LTC4412I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
- U3: MouserLink (none) -> https://www.mouser.at/ProductDetail/onsemi-Fairchild/FSUSB4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
- U4: MouserLink (none) -> https://www.mouser.at/ProductDetail/Olimex-Ltd/GL850G?qs=do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
- Y1: MouserLink (none) -> https://www.mouser.at/ProductDetail/ECS/ECS-120-18-4X-CKM?q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

Commit message: added mouser links to all components
Parts:
- C1: MouserLink (none) -> https://www.mouser.at/ProductDetail/Panasonic/EEU-FR1C101?q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
- C13, C2, C3, C8, C9: MouserLink (none) -> https://www.mouser.at/ProductDetail/TDK/C0603X5R1E104K030BB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
- C19: MouserLink (none) -> https://www.mouser.at/ProductDetail/KYOCERA-AVX/06033A330FA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
- L1, L2, L3, L4, L5, L6, L7: MouserLink (none) -> https://www.mouser.at/ProductDetail/Murata-Electronics/BLM1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
- R1, R2, R4, R9: MouserLink (none) -> https://www.mouser.at/ProductDetail/Panasonic/ERJ-UP3F5111V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
- R10, R5: MouserLink (none) -> https://www.mouser.at/ProductDetail/ROHM-Semiconductor/SDR0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
- R11: MouserLink (none) -> https://www.mouser.at/ProductDetail/YAGEO/RT0603FRE07100KL?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
- R12: MouserLink (none) -> https://www.mouser.at/ProductDetail/Panasonic/ERJ-3EKF6800V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
- R13, R6: MouserLink (none) -> https://www.mouser.at/ProductDetail/Panasonic/ERJ-3EKF1002V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
- R14: MouserLink (none) -> https://www.mouser.at/ProductDetail/YAGEO/RC0603JR-1347KL?q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
- R3: MouserLink (none) -> https://www.mouser.at/ProductDetail/ROHM-Semiconductor/SFR0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
- R7: MouserLink (none) -> https://www.mouser.at/ProductDetail/Vishay-Dale/CRCW060320K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
- R8: MouserLink (none) -> https://www.mouser.at/ProductDetail/Bourns/CR0603-FX-7870EL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
- SW1: MouserLink (none) -> https://www.mouser.at/ProductDetail/Chip-Quik/HDR100IMP40M-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
Changed lines of the file:
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@@
+      (effects (font (size 1.27 1.27)) hide)
+    )
+    (property "MouserLink" "https://www.mouser.at/ProductDetail/ROHM-Semiconductor/SDR03EZPF1004?qs=sGAEpiMZZMtlubZbdhIBIPTwcdbU5mXWm2PjMp1V47o%3D" (id 4) (at 66.04 97.79 0)
       (effects (font (size 1.27 1.27)) hide)
     )
@@
       (effects (font (size 1.27 1.27)) hide)
     )
+    (property "MouserLink" "https://www.mouser.at/ProductDetail/Murata-Electronics/BLM18KG601SH1D?qs=DXqDLUyyb5XOGozqLTtJZQ%3D%3D" (id 4) (at 255.27 60.96 90)
+      (effects (font (size 1.27 1.27)) hide)
+    )
     (pin "1")
     (pin "2")
@@
     )
     (property "Datasheet" "~" (id 3) (at 105.41 82.55 0)
+      (effects (font (size 1.27 1.27)) hide)
+    )
+    (property "MouserLink" "https://www.mouser.at/ProductDetail/Panasonic/ERJ-3EKF6800V?qs=sGAEpiMZZMtG0KNrPCHnjTg0x5DoQJ5PnxsrYk8gX6U%3D" (id 4) (at 105.41 82.55 90)
       (effects (font (size 1.27 1.27)) hide)
     )
@@
       (effects (font (size 1.27 1.27)) hide)
     )
+    (property "MouserLink" "https://www.mouser.at/ProductDetail/YAGEO/RT0603FRE07100KL?qs=sGAEpiMZZMtG0KNrPCHnjTg0x5DoQJ5PtfUThCgUIgQ%3D" (id 4) (at 257.81 34.29 0)
+      (effects (font (size 1.27 1.27)) hide)
+    )
     (pin "1")
     (pin "2")
@@
       (effects (font (size 1.27 1.27)) hide)
     )
+    (property "MouserLink" "https://www.mouser.at/ProductDetail/Bourns/CR0603-FX-7870ELF?qs=sGAEpiMZZMtG0KNrPCHnjfC2zYK6Lg3%2FtHnVIy8%252Bw4Y%3D" (id 4) (at 266.7 26.67 0)
+      (effects (font (size 1.27 1.27)) hide)
+    )
     (pin "1")
     (pin "2")
@@
     )
     (property "Datasheet" "~" (id 3) (at 190.5 29.21 0)
+      (effects (font (size 1.27 1.27)) hide)
+    )
+    (property "MouserLink" "https://www.mouser.at/ProductDetail/Panasonic/ERJ-3EKF1002V?qs=sGAEpiMZZMtG0KNrPCHnjWXb3yLuGJ273jbET5rTjY4%3D" (id 4) (at 190.5 29.21 0)
       (effects (font (size 1.27 1.27)) hide)
     )
@@
       (effects (font (size 1.27 1.27)) hide)
     )
+    (property "MouserLink" "https://www.mouser.at/ProductDetail/KYOCERA-AVX/06033A330FAT2A?qs=3M9tbN%252BqtAYbLVCRqESR2w%3D%3D" (id 4) (at 189.23 62.23 0)
+      (effects (font (size 1.27 1.27)) hide)
+    )
     (pin "1")
     (pin "2")
@@
     )
     (property "Datasheet" "~" (id 3) (at 237.49 99.06 0)
+      (effects (font (size 1.27 1.27)) hide)
+    )
+    (property "MouserLink" "https://www.mouser.at/ProductDetail/Murata-Electronics/BLM18KG601SH1D?qs=DXqDLUyyb5XOGozqLTtJZQ%3D%3D" (id 4) (at 237.49 99.06 90)
       (effects (font (size 1.27 1.27)) hide)
     )
@@
       (effects (font (size 1.27 1.27)) hide)
     )
+    (property "MouserLink" "https://www.mouser.at/ProductDetail/Murata-Electronics/BLM18KG601SH1D?qs=DXqDLUyyb5XOGozqLTtJZQ%3D%3D" (id 4) (at 237.49 134.62 90)
+      (effects (font (size 1.27 1.27)) hide)
+    )
     (pin "1")
     (pin "2")
@@
     )
     (property "Datasheet" "~" (id 3) (at 69.85 186.69 0)
+      (effects (font (size 1.27 1.27)) hide)
+    )
+    (property "MouserLink" "https://www.mouser.at/ProductDetail/ROHM-Semiconductor/SFR03EZPJ474?qs=sGAEpiMZZMtG0KNrPCHnjRpfexHZHoPIzYZevmk2KwpWeAu27XnBqA%3D%3D" (id 4) (at 69.85 186.69 90)
       (effects (font (size 1.27 1.27)) hide)
     )
@@
       (effects (font (size 1.27 1.27)) hide)
     )
+    (property "MouserLink" "https://www.mouser.at/ProductDetail/Vishay-Dale/CRCW060320K0JNEB?qs=sGAEpiMZZMtG0KNrPCHnjUwx9ESGNTAnYOn3oZE%2FWBU%3D" (id 4) (at 190.5 40.64 0)
+      (effects (font (size 1.27 1.27)) hide)
+    )
     (pin "1")
     (pin "2")
@@
     )
     (property "Datasheet" "~" (id 3) (at 130.81 44.45 0)
+      (effects (font (size 1.27 1.27)) hide)
+    )
+    (property "MouserLink" "https://www.mouser.at/ProductDetail/Chip-Quik/HDR100IMP40M-G-V-TH?qs=Wj%2FVkw3K%252BMBASWNGaQOKpg%3D%3D" (id 4) (at 130.81 44.45 0)
       (effects (font (size 1.27 1.27)) hide)
     )
@@
       (effects (font (size 1.27 1.27)) hide)
     )
+    (property "MouserLink" "https://www.mouser.at/ProductDetail/TDK/C0603X5R1E104K030BB?qs=6JAMGB%252BEdkw5r7LrYHn6NA%3D%3D" (id 4) (at 77.47 168.91 0)
+      (effects (font (size 1.27 1.27)) hide)
+    )
     (pin "1")
     (pin "2")
@@
       (effects (font (size 1.27 1.27)) hide)
     )
+    (property "MouserLink" "https://www.mouser.at/ProductDetail/Panasonic/EEU-FR1C101?qs=ob%252BdNz2%252BYEhUA1aQKNasqg%3D%3D" (id 4) (at 72.39 168.91 0)
+      (effects (font (size 1.27 1.27)) hide)
+    )
     (pin "1")
     (pin "2")
@@
       (effects (font (size 1.27 1.27)) hide)
     )
+    (property "MouserLink" "https://www.mouser.at/ProductDetail/Murata-Electronics/BLM18KG601SH1D?qs=DXqDLUyyb5XOGozqLTtJZQ%3D%3D" (id 4) (at 82.55 132.08 0)
+      (effects (font (size 1.27 1.27)) hide)
+    )
     (pin "1")
     (pin "2")
@@
       (effects (font (size 1.27 1.27)) hide)
     )
+    (property "MouserLink" "https://www.mouser.at/ProductDetail/TDK/C0603X5R1E104K030BB?qs=6JAMGB%252BEdkw5r7LrYHn6NA%3D%3D" (id 4) (at 158.75 109.22 0)
+      (effects (font (size 1.27 1.27)) hide)
+    )
     (pin "1")
     (pin "2")
@@
       (effects (font (size 1.27 1.27)) hide)
     )
+    (property "MouserLink" "https://www.mouser.at/ProductDetail/Panasonic/ERJ-UP3F5111V?qs=GedFDFLaBXH0bh5FmrY8eQ%3D%3D" (id 4) (at 15.24 74.93 0)
+      (effects (font (size 1.27 1.27)) hide)
+    )
     (pin "1")
     (pin "2")
@@
       (effects (font (size 1.27 1.27)) hide)
     )
+    (property "MouserLink" "https://www.mouser.at/ProductDetail/TDK/C0603X5R1E104K030BB?qs=6JAMGB%252BEdkw5r7LrYHn6NA%3D%3D" (id 4) (at 167.64 91.44 0)
+      (effects (font (size 1.27 1.27)) hide)
+    )
     (pin "1")
     (pin "2")
@@
     )
     (property "Datasheet" "~" (id 3) (at 226.06 40.64 0)
+      (effects (font (size 1.27 1.27)) hide)
+    )
+    (property "MouserLink" "https://www.mouser.at/ProductDetail/TDK/C0603X5R1E104K030BB?qs=6JAMGB%252BEdkw5r7LrYHn6NA%3D%3D" (id 4) (at 226.06 40.64 0)
       (effects (font (size 1.27 1.27)) hide)
     )
@@
       (effects (font (size 1.27 1.27)) hide)
     )
+    (property "MouserLink" "https://www.mouser.at/ProductDetail/ROHM-Semiconductor/SDR03EZPF1004?qs=sGAEpiMZZMtlubZbdhIBIPTwcdbU5mXWm2PjMp1V47o%3D" (id 4) (at 66.04 142.24 0)
+      (effects (font (size 1.27 1.27)) hide)
+    )
     (pin "1")
     (pin "2")
@@
     )
     (property "Datasheet" "~" (id 3) (at 77.47 69.85 0)
+      (effects (font (size 1.27 1.27)) hide)
+    )
+    (property "MouserLink" "https://www.mouser.at/ProductDetail/Panasonic/ERJ-UP3F5111V?qs=GedFDFLaBXH0bh5FmrY8eQ%3D%3D" (id 4) (at 77.47 69.85 0)
       (effects (font (size 1.27 1.27)) hide)
     )
@@
       (effects (font (size 1.27 1.27)) hide)
     )
+    (property "MouserLink" "https://www.mouser.at/ProductDetail/Panasonic/ERJ-UP3F5111V?qs=GedFDFLaBXH0bh5FmrY8eQ%3D%3D" (id 4) (at 77.47 114.3 0)
+      (effects (font (size 1.27 1.27)) hide)
+    )
     (pin "1")
     (pin "2")
@@
     )
     (property "Datasheet" "~" (id 3) (at 118.11 22.86 0)
+      (effects (font (size 1.27 1.27)) hide)
+    )
+    (property "MouserLink" "https://www.mouser.at/ProductDetail/TDK/C0603X5R1E104K030BB?qs=6JAMGB%252BEdkw5r7LrYHn6NA%3D%3D" (id 4) (at 118.11 22.86 0)
       (effects (font (size 1.27 1.27)) hide)
     )
@@
       (effects (font (size 1.27 1.27)) hide)
     )
+    (property "MouserLink" "https://www.mouser.at/ProductDetail/Murata-Electronics/BLM18KG601SH1D?qs=DXqDLUyyb5XOGozqLTtJZQ%3D%3D" (id 4) (at 237.49 130.81 90)
+      (effects (font (size 1.27 1.27)) hide)
+    )
     (pin "1")
     (pin "2")
@@
     )
     (property "Datasheet" "~" (id 3) (at 237.49 95.25 0)
+      (effects (font (size 1.27 1.27)) hide)
+    )
+    (property "MouserLink" "https://www.mouser.at/ProductDetail/Murata-Electronics/BLM18KG601SH1D?qs=DXqDLUyyb5XOGozqLTtJZQ%3D%3D" (id 4) (at 237.49 95.25 90)
       (effects (font (size 1.27 1.27)) hide)
     )
@@
       (effects (font (size 1.27 1.27)) hide)
     )
+    (property "MouserLink" "https://www.mouser.at/ProductDetail/Murata-Electronics/BLM18KG601SH1D?qs=DXqDLUyyb5XOGozqLTtJZQ%3D%3D" (id 4) (at 82.55 87.63 0)
+      (effects (font (size 1.27 1.27)) hide)
+    )
     (pin "1")
     (pin "2")
@@
       (effects (font (size 1.27 1.27)) hide)
     )
+    (property "MouserLink" "https://www.mouser.at/ProductDetail/Panasonic/ERJ-3EKF1002V?qs=sGAEpiMZZMtG0KNrPCHnjWXb3yLuGJ273jbET5rTjY4%3D" (id 4) (at 217.17 29.21 0)
+      (effects (font (size 1.27 1.27)) hide)
+    )
     (pin "1")
     (pin "2")
@@
     )
     (property "Datasheet" "~" (id 3) (at 15.24 119.38 0)
+      (effects (font (size 1.27 1.27)) hide)
+    )
+    (property "MouserLink" "https://www.mouser.at/ProductDetail/Panasonic/ERJ-UP3F5111V?qs=GedFDFLaBXH0bh5FmrY8eQ%3D%3D" (id 4) (at 15.24 119.38 0)
       (effects (font (size 1.27 1.27)) hide)
     )
@@
       (effects (font (size 1.27 1.27)) hide)
     )
+    (property "MouserLink" "https://www.mouser.at/ProductDetail/YAGEO/RC0603JR-1347KL?qs=sGAEpiMZZMtG0KNrPCHnjTg0x5DoQJ5P5TUM9gGimVE%3D" (id 4) (at 217.17 40.64 0)
+      (effects (font (size 1.27 1.27)) hide)
+    )

Commit message: updated link to 100nF caps
Parts:
- C11, C12, C13, C14, C17, C18, C2, C21, C3, C4, C5, C8, C9: MouserLink https://www.mouser.at/ProductDetail/TDK/C0603X5R1E104K030BB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 -> https://www.mouser.at/ProductDetail/TDK/CGA3E2X5R1H104M080A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
Changed lines of the file:
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@@
       (effects (font (size 1.27 1.27)) hide)
     )
-    (property "MouserLink" "https://www.mouser.at/ProductDetail/TDK/C0603X5R1E104K030BB?qs=6JAMGB%252BEdkw5r7LrYHn6NA%3D%3D" (id 4) (at 243.84 91.44 0)
+    (property "MouserLink" "https://www.mouser.at/ProductDetail/TDK/CGA3E2X5R1H104M080AA?qs=xLDY6iXSiQbtbwBJJW9HMQ%3D%3D" (id 4) (at 243.84 91.44 0)
       (effects (font (size 1.27 1.27)) hide)
     )
@@
       (effects (font (size 1.27 1.27)) hide)
     )
-    (property "MouserLink" "https://www.mouser.at/ProductDetail/TDK/C0603X5R1E104K030BB?qs=6JAMGB%252BEdkw5r7LrYHn6NA%3D%3D" (id 4) (at 243.84 64.77 0)
+    (property "MouserLink" "https://www.mouser.at/ProductDetail/TDK/CGA3E2X5R1H104M080AA?qs=xLDY6iXSiQbtbwBJJW9HMQ%3D%3D" (id 4) (at 243.84 64.77 0)
       (effects (font (size 1.27 1.27)) hide)
     )
@@
       (effects (font (size 1.27 1.27)) hide)
     )
-    (property "MouserLink" "https://www.mouser.at/ProductDetail/TDK/C0603X5R1E104K030BB?qs=6JAMGB%252BEdkw5r7LrYHn6NA%3D%3D" (id 4) (at 238.76 64.77 0)
+    (property "MouserLink" "https://www.mouser.at/ProductDetail/TDK/CGA3E2X5R1H104M080AA?qs=xLDY6iXSiQbtbwBJJW9HMQ%3D%3D" (id 4) (at 238.76 64.77 0)
       (effects (font (size 1.27 1.27)) hide)
     )
@@
       (effects (font (size 1.27 1.27)) hide)
     )
-    (property "MouserLink" "https://www.mouser.at/ProductDetail/TDK/C0603X5R1E104K030BB?qs=6JAMGB%252BEdkw5r7LrYHn6NA%3D%3D" (id 4) (at 248.92 64.77 0)
+    (property "MouserLink" "https://www.mouser.at/ProductDetail/TDK/CGA3E2X5R1H104M080AA?qs=xLDY6iXSiQbtbwBJJW9HMQ%3D%3D" (id 4) (at 248.92 64.77 0)
       (effects (font (size 1.27 1.27)) hide)
     )
@@
       (effects (font (size 1.27 1.27)) hide)
     )
-    (property "MouserLink" "https://www.mouser.at/ProductDetail/TDK/C0603X5R1E104K030BB?qs=6JAMGB%252BEdkw5r7LrYHn6NA%3D%3D" (id 4) (at 243.84 102.87 0)
+    (property "MouserLink" "https://www.mouser.at/ProductDetail/TDK/CGA3E2X5R1H104M080AA?qs=xLDY6iXSiQbtbwBJJW9HMQ%3D%3D" (id 4) (at 243.84 102.87 0)
       (effects (font (size 1.27 1.27)) hide)
     )
@@
       (effects (font (size 1.27 1.27)) hide)
     )
-    (property "MouserLink" "https://www.mouser.at/ProductDetail/TDK/C0603X5R1E104K030BB?qs=6JAMGB%252BEdkw5r7LrYHn6NA%3D%3D" (id 4) (at 77.47 168.91 0)
+    (property "MouserLink" "https://www.mouser.at/ProductDetail/TDK/CGA3E2X5R1H104M080AA?qs=xLDY6iXSiQbtbwBJJW9HMQ%3D%3D" (id 4) (at 77.47 168.91 0)
       (effects (font (size 1.27 1.27)) hide)
     )
@@
       (effects (font (size 1.27 1.27)) hide)
     )
-    (property "MouserLink" "https://www.mouser.at/ProductDetail/TDK/C0603X5R1E104K030BB?qs=6JAMGB%252BEdkw5r7LrYHn6NA%3D%3D" (id 4) (at 158.75 109.22 0)
+    (property "MouserLink" "https://www.mouser.at/ProductDetail/TDK/CGA3E2X5R1H104M080AA?qs=xLDY6iXSiQbtbwBJJW9HMQ%3D%3D" (id 4) (at 158.75 109.22 0)
       (effects (font (size 1.27 1.27)) hide)
     )
@@
       (effects (font (size 1.27 1.27)) hide)
     )
-    (property "MouserLink" "https://www.mouser.at/ProductDetail/TDK/C0603X5R1E104K030BB?qs=6JAMGB%252BEdkw5r7LrYHn6NA%3D%3D" (id 4) (at 167.64 91.44 0)
+    (property "MouserLink" "https://www.mouser.at/ProductDetail/TDK/CGA3E2X5R1H104M080AA?qs=xLDY6iXSiQbtbwBJJW9HMQ%3D%3D" (id 4) (at 167.64 91.44 0)
       (effects (font (size 1.27 1.27)) hide)
     )
@@
       (effects (font (size 1.27 1.27)) hide)
     )
-    (property "MouserLink" "https://www.mouser.at/ProductDetail/TDK/C0603X5R1E104K030BB?qs=6JAMGB%252BEdkw5r7LrYHn6NA%3D%3D" (id 4) (at 226.06 40.64 0)
+    (property "MouserLink" "https://www.mouser.at/ProductDetail/TDK/CGA3E2X5R1H104M080AA?qs=xLDY6iXSiQbtbwBJJW9HMQ%3D%3D" (id 4) (at 226.06 40.64 0)
       (effects (font (size 1.27 1.27)) hide)
     )
@@
       (effects (font (size 1.27 1.27)) hide)
     )
-    (property "MouserLink" "https://www.mouser.at/ProductDetail/TDK/C0603X5R1E104K030BB?qs=6JAMGB%252BEdkw5r7LrYHn6NA%3D%3D" (id 4) (at 243.84 138.43 0)
+    (property "MouserLink" "https://www.mouser.at/ProductDetail/TDK/CGA3E2X5R1H104M080AA?qs=xLDY6iXSiQbtbwBJJW9HMQ%3D%3D" (id 4) (at 243.84 138.43 0)
       (effects (font (size 1.27 1.27)) hide)
     )
@@
       (effects (font (size 1.27 1.27)) hide)
     )
-    (property "MouserLink" "https://www.mouser.at/ProductDetail/TDK/C0603X5R1E104K030BB?qs=6JAMGB%252BEdkw5r7LrYHn6NA%3D%3D" (id 4) (at 118.11 22.86 0)
+    (property "MouserLink" "https://www.mouser.at/ProductDetail/TDK/CGA3E2X5R1H104M080AA?qs=xLDY6iXSiQbtbwBJJW9HMQ%3D%3D" (id 4) (at 118.11 22.86 0)
       (effects (font (size 1.27 1.27)) hide)
     )
@@
       (effects (font (size 1.27 1.27)) hide)
     )
-    (property "MouserLink" "https://www.mouser.at/ProductDetail/TDK/C0603X5R1E104K030BB?qs=6JAMGB%252BEdkw5r7LrYHn6NA%3D%3D" (id 4) (at 233.68 64.77 0)
+    (property "MouserLink" "https://www.mouser.at/ProductDetail/TDK/CGA3E2X5R1H104M080AA?qs=xLDY6iXSiQbtbwBJJW9HMQ%3D%3D" (id 4) (at 233.68 64.77 0)
       (effects (font (size 1.27 1.27)) hide)
     )
@@
       (effects (font (size 1.27 1.27)) hide)
     )
-    (property "MouserLink" "https://www.mouser.at/ProductDetail/TDK/C0603X5R1E104K030BB?qs=6JAMGB%252BEdkw5r7LrYHn6NA%3D%3D" (id 4) (at 243.84 127 0)
-      (effects (font (size 1.27 1.27)) hide)
-    )
+    (property "MouserLink" "https://www.mouser.at/ProductDetail/TDK/CGA3E2X5R1H104M080AA?qs=xLDY6iXSiQbtbwBJJW9HMQ%3D%3D" (id 4) (at 243.84 127 0)
+      (effects (font (size 1.27 1.27)) hide)
+    )
